File: pcb/CANdiy-Shield_v13.sch (EAGLE design)
At the start: 57 parts, among them IC2 MCP2551SO8, Q1 16MHz, U1 UNO_ISP

Commit message: cleaned up schematics and layout
Changed lines of the file:
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@@
 <setting verticaltext="up"/>
 </settings>
-<grid distance="0.1" unitdist="inch" unit="inch" style="lines" multiple="1" display="no" altdistance="0.01" altunitdist="inch" altunit="inch"/>
+<grid distance="0.05" unitdist="inch" unit="inch" style="lines" multiple="1" display="yes" altdistance="0.025" altunitdist="inch" altunit="inch"/>
 <layers>
 <layer number="1" name="Top" color="4" fill="1" visible="no" active="no"/>
@@
 </classes>
 <parts>
-<part name="FRAME1" library="frames" deviceset="A4L-LOC" device=""/>
 <part name="GND4" library="supply1" deviceset="GND" device=""/>
 <part name="LOGO2" library="OSHW" deviceset="OSHW_LOGO_6MIL" device="X0100-NT"/>
@@
 <part name="Q1" library="crystal" deviceset="SMD_OSC" device="2" value="16MHz"/>
 <part name="IC1" library="can" deviceset="MCP2515" device="ST"/>
+<part name="FRAME1" library="we-symbol" deviceset="FRAME-A4L" device=""/>
 </parts>
 <sheets>
 <sheet>
 <plain>
-<text x="161.29" y="34.29" size="1.27" layer="95">Released under the Creative Commons Attribution Share-Alike License</text>
-<text x="161.29" y="31.75" size="1.27" layer="95">http://creativecommons.org/licenses/by-sa/4.0/</text>
-<text x="161.29" y="27.94" size="1.27" layer="95">Designed by Stephan Watterott (Watterott electronic)</text>
+<text x="162.56" y="21.59" size="1.27" layer="95">Released under the Creative Commons Attribution Share-Alike License</text>
+<text x="162.56" y="19.05" size="1.27" layer="95">http://creativecommons.org/licenses/by-sa/4.0/</text>
+<text x="162.56" y="15.24" size="1.27" layer="95">Designed by Stephan Watterott (Watterott electronic)</text>
 <text x="45.72" y="133.35" size="3.81" layer="250">Arduino</text>
 <text x="167.64" y="121.92" size="1.6764" layer="95">F1</text>
@@
 <text x="132.08" y="139.7" size="1.778" layer="94">JP3 - Short for GND connection (required for Railuino)</text>
 <text x="132.08" y="142.24" size="1.778" layer="94">JP2 - Short for VIN connection (required for Railuino)</text>
-<text x="161.29" y="25.4" size="1.27" layer="95">Based on the work of Jörg Pleumann</text>
+<text x="162.56" y="12.7" size="1.27" layer="95">Based on the work of Jörg Pleumann</text>
 <text x="119.38" y="101.6" size="3.81" layer="250">CAN Controller</text>
 <text x="166.37" y="101.6" size="3.81" layer="250">CAN Transceiver</text>
 </plain>
 <instances>
-<instance part="FRAME1" gate="G$1" x="0" y="0" smashed="yes">
-<attribute name="DRAWING_NAME" x="217.17" y="15.24" size="2.54" layer="94" font="vector"/>
-<attribute name="LAST_DATE_TIME" x="217.17" y="10.16" size="2.286" layer="94" font="vector"/>
-<attribute name="SHEET" x="230.505" y="5.08" size="2.54" layer="94" font="vector"/>
-</instance>
 <instance part="GND4" gate="1" x="113.03" y="129.54" smashed="yes" rot="R90">
 <attribute name="VALUE" x="115.57" y="127" size="1.778" layer="96" rot="R90"/>
 </instance>
-<instance part="LOGO2" gate="G$1" x="201.93" y="19.05"/>
+<instance part="LOGO2" gate="G$1" x="198.12" y="7.62"/>
 <instance part="GND14" gate="1" x="24.13" y="101.6" smashed="yes" rot="R270">
 <attribute name="VALUE" x="21.59" y="104.14" size="1.778" layer="96" rot="R270"/>
@@
 <attribute name="VALUE" x="111.125" y="29.21" size="1.778" layer="96" rot="R90"/>
 </instance>
-<instance part="U$1" gate="G$1" x="201.93" y="11.43"/>
+<instance part="U$1" gate="G$1" x="208.28" y="7.62"/>
 <instance part="C7" gate="G$1" x="143.51" y="123.19"/>
 <instance part="D1" gate="G$1" x="157.48" y="125.73" smashed="yes" rot="R180">
@@
 <attribute name="VALUE" x="146.05" y="113.03" size="1.778" layer="96" rot="MR0"/>
 </instance>
-<instance part="X_2" gate="G$1" x="166.37" y="11.43"/>
-<instance part="X_1" gate="G$1" x="173.99" y="11.43"/>
+<instance part="X_2" gate="G$1" x="165.1" y="7.62"/>
+<instance part="X_1" gate="G$1" x="170.18" y="7.62"/>
 <instance part="U1" gate="G$1" x="54.61" y="96.52"/>
 <instance part="5V" gate="P" x="25.4" y="114.3" smashed="yes">
@@
 <instance part="IC1" gate="D" x="137.16" y="81.28"/>
 <instance part="IC1" gate="P" x="21.59" y="25.4"/>
+<instance part="FRAME1" gate="G$1" x="0" y="0"/>
 </instances>
 <busses>
