File: pcb/CANdiy-Shield_v20.sch (EAGLE design)
At the start: 59 parts, among them IC1 MCP2515, IC2 MCP2562, Q1 16MHz, U1 UNO_ISP, X1 PASSER, X2 PASSER, X3 PASSER

Commit message: cleaned up schematics and layout
Changed lines of the file:
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@@
 <setting verticaltext="up"/>
 </settings>
-<grid distance="0.1" unitdist="inch" unit="inch" style="lines" multiple="1" display="no" altdistance="0.01" altunitdist="inch" altunit="inch"/>
+<grid distance="0.05" unitdist="inch" unit="inch" style="lines" multiple="1" display="yes" altdistance="0.025" altunitdist="inch" altunit="inch"/>
 <layers>
 <layer number="1" name="Top" color="4" fill="1" visible="no" active="no"/>
@@
 </classes>
 <parts>
-<part name="FRAME1" library="frames" deviceset="A4L-LOC" device=""/>
 <part name="GND4" library="supply1" deviceset="GND" device=""/>
 <part name="LOGO2" library="OSHW" deviceset="OSHW_LOGO_6MIL" device="X0100-NT"/>
@@
 <part name="X3" library="we-symbol" deviceset="PASSER" device=""/>
 <part name="LOGO1" library="we-symbol" deviceset="LOGO" device="-SPARK_PLACE"/>
+<part name="FRAME1" library="we-symbol" deviceset="FRAME-A4L" device=""/>
 </parts>
 <sheets>
 <sheet>
 <plain>
-<text x="161.29" y="31.75" size="1.27" layer="95">Released under the Creative Commons Attribution Share-Alike License</text>
-<text x="161.29" y="29.21" size="1.27" layer="95">http://creativecommons.org/licenses/by-sa/4.0/</text>
-<text x="161.29" y="25.4" size="1.27" layer="95">Designed by Stephan Watterott (Watterott electronic)</text>
+<text x="162.56" y="21.59" size="1.27" layer="95">Released under the Creative Commons Attribution Share-Alike License</text>
+<text x="162.56" y="19.05" size="1.27" layer="95">http://creativecommons.org/licenses/by-sa/4.0/</text>
+<text x="162.56" y="15.24" size="1.27" layer="95">Designed by Stephan Watterott (Watterott electronic)</text>
 <text x="43.18" y="135.89" size="3.81" layer="95">Arduino</text>
 <text x="223.52" y="96.52" size="2.54" layer="94">CAN Termination</text>
@@
 </plain>
 <instances>
-<instance part="FRAME1" gate="G$1" x="0" y="0" smashed="yes">
-<attribute name="DRAWING_NAME" x="217.17" y="15.24" size="2.54" layer="94" font="vector"/>
-<attribute name="LAST_DATE_TIME" x="217.17" y="10.16" size="2.286" layer="94" font="vector"/>
-<attribute name="SHEET" x="230.505" y="5.08" size="2.54" layer="94" font="vector"/>
-</instance>
 <instance part="GND4" gate="1" x="111.76" y="129.54" smashed="yes" rot="R90">
 <attribute name="VALUE" x="114.3" y="127" size="1.778" layer="96" rot="R90"/>
 </instance>
-<instance part="LOGO2" gate="G$1" x="203.2" y="10.16"/>
+<instance part="LOGO2" gate="G$1" x="187.96" y="7.62"/>
 <instance part="GND14" gate="1" x="24.13" y="106.68" smashed="yes" rot="R270">
 <attribute name="VALUE" x="21.59" y="109.22" size="1.778" layer="96" rot="R270"/>
@@
 <attribute name="VALUE" x="131.445" y="25.4" size="1.778" layer="96" rot="R90"/>
 </instance>
-<instance part="U$1" gate="G$1" x="172.72" y="10.16"/>
+<instance part="U$1" gate="G$1" x="198.12" y="7.62"/>
 <instance part="D1" gate="G$1" x="163.83" y="125.73" smashed="yes" rot="R180">
 <attribute name="NAME" x="163.83" y="122.7074" size="1.778" layer="95" rot="R180"/>
@@
 <attribute name="VALUE" x="100.965" y="113.03" size="1.778" layer="96" rot="R90"/>
 </instance>
-<instance part="X1" gate="G$1" x="170.18" y="19.05"/>
-<instance part="X2" gate="G$1" x="185.42" y="19.05"/>
-<instance part="X3" gate="G$1" x="200.66" y="19.05"/>
-<instance part="LOGO1" gate="G$1" x="187.96" y="10.16"/>
+<instance part="X1" gate="G$1" x="165.1" y="7.62"/>
+<instance part="X2" gate="G$1" x="170.18" y="7.62"/>
+<instance part="X3" gate="G$1" x="175.26" y="7.62"/>
+<instance part="LOGO1" gate="G$1" x="208.28" y="7.62"/>
+<instance part="FRAME1" gate="G$1" x="0" y="0"/>
 </instances>
 <busses>
